File: hardware/nrf52.kicad_sch (KiCad schematic)
At the start: 70 parts, among them J1 Conn_01x20, J2 USB_C_Receptacle_USB2.0_14P, J3 Conn_01x10, J4 Conn_01x20, J6 LiPo, Q1 Si1308EDL, Q2 AO3401A, SW1 SW_Push, U1 nRF52840, U2 Conn_Eink_1.9"_Generic, U3 SRV05-4, U4 TP4057, U5 HE9073A33M5R, Y1 32MHz 12pF, Y2 32.768kHz 12.5pF

Commit message: Stash
Parts:
- removed C23, C25, C26, C28, C30, C31, C32, C37, C7: 1uF, Capacitor_SMD:C_0402_1005Metric, symbol Device:C
- removed C24, C33: 1uF, Capacitor_SMD:C_0402_1005Metric, symbol Device:C_Small
- removed C27, C29: 4.7uF, Capacitor_SMD:C_0402_1005Metric, symbol Device:C
- removed D1, D2, D3: MBR0530, Diode_SMD:D_SOD-123, symbol Diode:MBR0530
- removed J6: LiPo, nrf52:HCTL_JST_PH_HC-PH-2AWT-B_2P, symbol Connector_Generic_MountingPin:Conn_01x02_MountingPin
- removed L6: 47uH 500mA, Inductor_SMD:L_APV_ANR3015, symbol Device:L
- removed Q1: Si1308EDL, Package_TO_SOT_SMD:SOT-323_SC-70, symbol Transistor_FET:Si1308EDL
- removed R12: 2.2R, Resistor_SMD:R_0402_1005Metric, symbol Device:R
- removed R13: 100k, Resistor_SMD:R_0402_1005Metric, symbol Device:R
- removed U2: Conn_Eink_1.9"_Generic, nrf52:HCTL_HC-FPC-05-09-24RLTAG-1MP_P0.5mm_Horizontal, symbol PCM_ckl-misc:Conn_Eink_1.9{dblquote}_Generic
- added D6, D7: LED, LED_SMD:LED_0402_1005Metric, symbol Device:LED
- added JP1: CUT, PCM_ckl-misc:SolderJumper-2_Bridged_Pad_Small, symbol Jumper:SolderJumper_2_Bridged
- added R11, R8: 1.5k, Resistor_SMD:R_0402_1005Metric, symbol Device:R
- C11, C17: footprint Capacitor_SMD:C_0603_1608Metric -> Capacitor_SMD:C_0402_1005Metric; LCSC Part # C15849 -> C7472946
- C13, C15, C16: LCSC Part # C19666 -> C380325
- J2: Position Offset (none) -> -1.775,0
- R5, R6: LCSC Part # C105872 -> C2906874
- U1: FT Rotation Offset (none) -> -90
- U3: FT Rotation Offset (none) -> 90
Connections:
- net +3V3: now also JP1.2 (B)
- net P0.17: now also D7.1 (K)
- net P0.18: now also D6.1 (K)
- new net: JP1.1 (A), R11.1, R8.1
- new net: D6.2 (A), R8.2
- new net: D7.2 (A), R11.2
- no-connect marks 8 -> 6

Commit message: Stash
Parts:
- added C23, C25, C26, C28, C30, C31, C32, C37, C7: 1uF, Capacitor_SMD:C_0402_1005Metric, symbol Device:C
- added C24, C33: 1uF, Capacitor_SMD:C_0402_1005Metric, symbol Device:C_Small
- added C27, C29: 4.7uF, Capacitor_SMD:C_0402_1005Metric, symbol Device:C
- added D1, D2, D3: MBR0530, Diode_SMD:D_SOD-123, symbol Diode:MBR0530
- added J6: LiPo, nrf52:HCTL_JST_PH_HC-PH-2AWT-B_2P, symbol Connector_Generic_MountingPin:Conn_01x02_MountingPin
- added L6: 47uH 500mA, Inductor_SMD:L_APV_ANR3015, symbol Device:L
- added Q1: Si1308EDL, Package_TO_SOT_SMD:SOT-323_SC-70, symbol Transistor_FET:Si1308EDL
- added R12: 2.2R, Resistor_SMD:R_0402_1005Metric, symbol Device:R
- added R13: 1M, Resistor_SMD:R_0402_1005Metric, symbol Device:R
- added U2: Conn_Eink_1.9"_Generic, nrf52:HCTL_HC-FPC-05-09-24RLTAG-1MP_P0.5mm_Horizontal, symbol PCM_ckl-misc:Conn_Eink_1.9{dblquote}_Generic
Connections:
- net +3V3: now also C23.1, C29.1, L6.1, U2.15 (VDDIO), U2.16 (VCI)
- net +BATT: now also C7.1, J6.2 (Pin_2)
- net BUSY: now also U2.9 (BUSY)
- net CLK: now also U2.13 (SCL)
- net GND: now also C23.2, C24.2, C25.2, C26.2, C28.2, C29.2, C30.2, C31.2, C32.2, C33.2, C37.2, C7.2, D2.1 (K), J6.1 (Pin_1), J6.MP (MountPin), R12.2, R13.1, U2.17 (VSS), U2.8 (BS1), U2.MP (SHIELD)
- net MOSI: now also U2.14 (SDA)
- net ~{CS}: now also U2.12 (~{CS})
- net ~{D/C}: now also U2.11 (~{D/C})
- net ~{RES}: now also U2.10 (~{RST})
- new net: C27.1, D1.1 (K), D2.2 (A)
- new net: C27.2, D3.2 (A), L6.2, Q1.3 (D)
- new net: C24.1, U2.4 (VGL/NC)
- new net: C32.1, U2.24 (VCOM)
- new net: C28.1, U2.20 (VSH1)
- new net: C30.1, U2.22 (VSL)
- new net: C37.1, U2.19 (VPP)
- new net: C25.1, U2.18 (VDD)
- new net: C33.1, U2.5 (VSH2)
- new net GDR: Q1.1 (G), R13.2, U2.2 (GDR)
- new net RESE: Q1.2 (S), R12.1, U2.3 (RESE)
- new net VGH: C31.1, D3.1 (K), U2.21 (VGH)
- new net VGL: C26.1, D1.2 (A), U2.23 (VGL)
- no-connect marks 6 -> 8
Other:
- moved on the sheet: D6, D7, JP1, R11, R8
