File: hardware/nrf52.kicad_pcb (KiCad board)
At the start: 4 copper layers, 59.7 x 30.5 mm, 70 parts, among them J1 Conn_01x20, J2 USB_C_Receptacle_USB2.0_14P, J3 Conn_01x10, J4 Conn_01x20, J6 LiPo, Q1 Si1308EDL, Q2 AO3401A, SW1 SW_Push, U1 nRF52840, U2 Conn_Eink_1.9"_Generic, U3 SRV05-4, U4 TP4057, U5 HE9073A33M5R, Y1 32MHz 12pF, Y2 32.768kHz 12.5pF

Commit message: Stash
Parts:
- added D6: LED, LED_SMD:LED_0402_1005Metric, F.Cu at (195.3, 132.7)
- added D7: LED, LED_SMD:LED_0402_1005Metric, F.Cu at (195.3, 133.7)
- added G*** (x2): LOGO, LOGO, F.Cu at (171.6, 144.4)
- added G*** (x3): LOGO, LOGO, B.Cu at (171.6, 144.4)
- added JP1: CUT, PCM_ckl-misc:SolderJumper-2_Bridged_Pad_Small, F.Cu at (197.7, 135.2)
- added R11: 1.5k, Resistor_SMD:R_0402_1005Metric, F.Cu at (197.2, 133.7)
- added R8: 1.5k, Resistor_SMD:R_0402_1005Metric, F.Cu at (197.2, 132.7)
- C11, C17: footprint Capacitor_SMD:C_0603_1608Metric -> Capacitor_SMD:C_0402_1005Metric
- R13: value 100k -> 1M
- moved C17 0.86 mm to (169.6, 149.8)
- moved C11 0.62 mm to (167.3, 151.9)
- moved L2 0.39 mm to (169.8, 151.3)
- moved L3 0.39 mm to (169.2, 152.5)
Routing:
- net +3V3: track 119.8 -> 125.6 mm
- net Net-(JP1-A): track 0.00 -> 1.90 mm
- net /P0.18: track 41.0 -> 42.3 mm, vias 1 -> 2
- net /P0.17: track 41.3 -> 42.4 mm, vias 1 -> 2
- net +BATT: track 35.9 -> 34.8 mm
- net Net-(D7-A): track 0.00 -> 0.90 mm
- net Net-(D6-A): track 0.00 -> 0.90 mm
- net /DEC4_6: track 12.8 -> 12.1 mm

Commit message: Stash
Parts:
- removed G*** (x5): LOGO, LOGO
